File: HFW8R-1STE1LF.kicad_pcb (KiCad board)
At the start: 2 copper layers, 30.5 x 25.4 mm, 1 part, among them J1 Conn_01x10_Male

Commit message: 3d rendering
Other:
- board size 30.5 x 25.4 mm -> 15.9 x 12.1 mm
Changed lines of the file:
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@@
   (general
     (thickness 1.6)
-    (drawings 5)
+    (drawings 4)
     (tracks 21)
     (zones 0)
@@
     (uvia_drill 0.1)
     (add_net "Net-(J1-Pad1)")
-    (add_net "Net-(J1-Pad10)")
     (add_net "Net-(J1-Pad2)")
     (add_net "Net-(J1-Pad3)")
     (add_net "Net-(J1-Pad4)")
-    (add_net "Net-(J1-Pad9)")
   )
   (module HFW8R-1STE1LF:HFW8R-1STE1LF (layer F.Cu)
@@
     )
   )
-  (gr_line (start 119.38 114.3) (end 119.38 101.6) (layer Edge.Cuts) (width 0.1))
-  (gr_line (start 149.86 114.3) (end 119.38 114.3) (layer Edge.Cuts) (width 0.1))
-  (gr_line (start 149.86 88.9) (end 149.86 114.3) (layer Edge.Cuts) (width 0.1))
-  (gr_line (start 119.38 88.9) (end 149.86 88.9) (layer Edge.Cuts) (width 0.1))
-  (gr_line (start 119.38 101.6) (end 119.38 88.9) (layer Edge.Cuts) (width 0.1))
+  (gr_line (start 126.365 104.775) (end 126.365 92.71) (layer Edge.Cuts) (width 0.1))
+  (gr_line (start 142.24 104.775) (end 126.365 104.775) (layer Edge.Cuts) (width 0.1))
+  (gr_line (start 142.24 92.71) (end 142.24 104.775) (layer Edge.Cuts) (width 0.1))
+  (gr_line (start 126.365 92.71) (end 142.24 92.71) (layer Edge.Cuts) (width 0.1))
   (segment (start 130.16 98.425) (end 130.16 95.265) (width 0.25) (layer F.Cu) (net 1))
   (segment (start 130.16 95.265) (end 131.445 93.98) (width 0.25) (layer F.Cu) (net 1))
